File: Keyboard.kicad_pcb (KiCad board)
At the start: 2 copper layers, 295.8 x 105.2 mm, 153 parts, among them J1 USB_C_Receptacle_USB2.0_14P, J4 Conn_01x03, SW1 SW_Push, SW10 SW_Push, SW11 SW_Push, SW12 SW_Push, SW13 SW_Push, SW14 SW_Push, SW15 SW_Push, SW16 SW_Push, SW17 SW_Push, SW18 SW_Push, SW19 SW_Push, SW2 SW_Push, SW20 SW_Push, SW21 SW_Push, SW22 SW_Push, SW23 SW_Push, SW24 SW_Push, SW25 SW_Push, SW26 SW_Push, SW27 SW_Push, SW28 SW_Push, SW29 SW_Push, SW3 SW_Push, SW30 SW_Push, SW31 SW_Push, SW32 SW_Push, SW33 SW_Push, SW34 SW_Push, SW35 SW_Push, SW36 SW_Push, SW37 SW_Push, SW38 SW_Push, SW39 SW_Push, SW4 SW_Push, SW40 SW_Push, SW41 SW_Push, SW42 SW_Push, SW43 SW_Push, SW44 SW_Push, SW45 SW_Push, SW46 SW_Push, SW47 SW_Push, SW48 SW_Push, SW49 SW_Push, SW5 SW_Push, SW50 SW_Push, SW51 SW_Push, SW52 SW_Push, SW53 SW_Push, SW54 SW_Push, SW55 SW_Push, SW56 SW_Push, SW57 SW_Push, SW58 SW_Push, SW59 SW_Push, SW6 SW_Push, SW60 SW_Push, SW61 SW_Push, SW62 SW_Push, SW7 SW_Push, SW8 SW_Push, SW9 SW_Push, U1 MCP1700x-330xxTT, U2 W25Q16JVUXIQ TR, U3 RP2040, Y1 12 MHz

Commit message: Fixed DRC
Parts:
- C8: moved to B.Cu
- moved C8 5.76 mm to (325.5, 82.0), turned to -90 degrees
- moved R7 1.33 mm to (326.6, 81.0)
- moved C17 0.94 mm to (332.2, 81.6)
- moved Y1 0.94 mm to (329.4, 81.6)
- moved C16 0.94 mm to (330.0, 79.2)
Routing:
- net GND: track 6.99 -> 20.9 mm, vias 14 -> 33
- net +3V3: track 56.2 -> 64.3 mm, vias 5 -> 6
- net Row 3: track 292.8 -> 294.1 mm
- net XOUT: track 3.84 -> 2.53 mm
- net Net-(C17-Pad2): track 6.40 -> 7.36 mm
- net Column 8: track 167.8 -> 168.7 mm
- net QSPI_SD1: track 6.15 -> 5.62 mm
